Commit message: fixed urdf file - still missing camera

File: catkin_ws/src/lakitu/urdf/lakitu.urdf (robot description, URDF)
Before this commit: robot lakitu, 4 links, 0 joints
Joints:
- added joint j1: type fixed, parent base_link, child airframe
- added joint j2: type fixed, parent airframe, child odroid
- added joint j3: type fixed, parent airframe, child pixracer_IMU

Commit message: got urdf and tf up and running in launch file, creating a node to publish poses to state machine

File: catkin_ws/src/lakitu/urdf/lakitu.urdf (robot description, URDF)
Before this commit: robot lakitu, 4 links, 3 joints
Links:
- added link camera; visual box size=0.1 0.1 0.1
Joints:
- added joint j4: type fixed, parent airframe, child camera
